File: 4_Isolated_CAN_node STM32G/4_Isolated_CAN_node STM32G.kicad_sch (KiCad schematic)
At the start: 6 parts, among them U1 STM32G431CBTx, U4 AP2112K-3.3, Y1 Crystal_GND24_Small

Commit message: progress in 4th project
Parts:
- added FL1: Filter_EMI_CommonMode, symbol Device:Filter_EMI_CommonMode
- added J1: USB_C_Receptacle_USB2.0_16P, symbol Connector:USB_C_Receptacle_USB2.0_16P
- added J2: DE9_Pins_MountingHoles, symbol Connector:DE9_Pins_MountingHoles
- added J3: Conn_01x04_Pin, symbol Connector:Conn_01x04_Pin
- added J4: Screw_Terminal_01x03, symbol Connector:Screw_Terminal_01x03
- added JP1: Jumper_2_Open, symbol Jumper:Jumper_2_Open
Connections:
- new net: J1.A1 (GND), J1.A12 (GND), J1.B1 (GND), J1.B12 (GND)
- new net: J1.A4 (VBUS), J1.A9 (VBUS), J1.B4 (VBUS), J1.B9 (VBUS)

Commit message: modify files
Parts:
- added C1, C2, C3, C4: C, symbol Device:C
- added D2: LED, symbol Device:LED
- added R1, R2, R3, R4, R5: R, symbol Device:R
Other:
- moved on the sheet: D1, FL1, J1, J2, J3, J4, JP1, U1, U2, U3, U4, Y1
