File: 4_Isolated_CAN_node STM32G (incomplete)/4_Isolated_CAN_node STM32G.kicad_sch (KiCad schematic)
At the start: 22 parts, among them J1 USB_C_Receptacle_USB2.0_16P, J2 DE9_Pins_MountingHoles, J3 Conn_01x04_Pin, J4 Screw_Terminal_01x03, U1 STM32G431CBTx, U4 AP2112K-3.3, Y1 Crystal_GND24_Small

Commit message: updated all the project also tag which one is complete and which one is not
Parts:
- added C5: 4.7nF, symbol Device:C
- added R6: 60, symbol Device:R
- R5: value R -> 60
Connections:
- net CAN_L: now reaches J2.2
- net CAN_L: now also J4.2 (Pin_2), R6.2
- net GND_ISO: now reaches J2.3
- net GND_ISO: now also J4.3 (Pin_3), C5.2
- net CAN_H: now reaches J2.7
- net CAN_H: now also J4.1 (Pin_1), JP1.2 (B)
- net at JP1.1 (A): now also R5.2
- net at R5.1: now also C5.1, R6.1
Other:
- moved on the sheet: JP1
